File: Hardware/Eagle/Schematic/NixieClock.brd (EAGLE design)
At the start: 297.8 x 112.7 mm, 16 parts, among them X0 5566-12, X1 5566-12, X2 5566-12, X3 5566-12, X4 5566-12, X5 5566-12

Commit message: Progress
Routing:
- net N$23: track 189.6 -> 197.7 mm, vias 1 -> 2
- net N$12: track 36.0 -> 37.8 mm
- net N$15: track 30.1 -> 29.4 mm

Commit message: Routed further chips' VCC and GND to the node's 3v3 and GND
Connections:
- new net N$44: BCD0.P$5, BCD1.P$5, SR0.P$10, SR0.P$16, U$1.3V3@2
- new net N$45: BCD0.P$12, BCD1.P$12, SR0.P$13, SR0.P$8, U$1.GND@3
- net N$13: now also U$1.3V3@0; no longer BCD0.P$5, BCD1.P$5, SR0.P$10, SR0.P$16, U$1.3V3@2
- net N$23: now also U$1.GND@0; no longer BCD0.P$12, BCD1.P$12, SR0.P$13, SR0.P$8, U$1.GND@3
Routing:
- net N$23: track 197.7 -> 37.2 mm, vias 2 -> 0
- net N$45: track 0.00 -> 156.8 mm, vias 0 -> 2
- net N$44: track 0.00 -> 136.4 mm
- net N$13: track 176.7 -> 143.0 mm
Changed lines of the file:
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@@
 <signal name="N$13">
 <contactref element="BCD3" pad="P$5"/>
+<contactref element="SR1" pad="P$10"/>
+<contactref element="BCD2" pad="P$5"/>
+<contactref element="SR1" pad="P$16"/>
+<contactref element="U$1" pad="3V3@0"/>
 <contactref element="BCD5" pad="P$5"/>
 <contactref element="SR2" pad="P$10"/>
 <contactref element="BCD4" pad="P$5"/>
 <contactref element="SR2" pad="P$16"/>
-<contactref element="BCD0" pad="P$5"/>
-<contactref element="SR0" pad="P$16"/>
-<contactref element="U$1" pad="3V3@2"/>
-<contactref element="BCD1" pad="P$5"/>
-<contactref element="SR0" pad="P$10"/>
-<contactref element="SR1" pad="P$10"/>
-<contactref element="BCD2" pad="P$5"/>
-<contactref element="SR1" pad="P$16"/>
-<wire x1="145.415" y1="71.755" x2="93.345" y2="71.755" width="0.1524" layer="1"/>
-<wire x1="93.345" y1="71.755" x2="90.805" y2="69.215" width="0.1524" layer="1"/>
-<wire x1="154.305" y1="80.645" x2="145.415" y2="71.755" width="0.1524" layer="1"/>
-<wire x1="75.565" y1="62.865" x2="76.835" y2="64.135" width="0.1524" layer="1"/>
-<wire x1="85.725" y1="64.135" x2="76.835" y2="64.135" width="0.1524" layer="1"/>
-<wire x1="90.805" y1="69.215" x2="85.725" y2="64.135" width="0.1524" layer="1"/>
-<wire x1="76.835" y1="57.785" x2="77.47" y2="58.42" width="0.1524" layer="1"/>
-<wire x1="77.47" y1="60.96" x2="75.565" y2="62.865" width="0.1524" layer="1"/>
-<wire x1="50.165" y1="69.215" x2="61.595" y2="57.785" width="0.1524" layer="1"/>
-<wire x1="61.595" y1="57.785" x2="76.835" y2="57.785" width="0.1524" layer="1"/>
-<wire x1="77.47" y1="58.42" x2="77.47" y2="60.96" width="0.1524" layer="1"/>
-<wire x1="50.165" y1="69.215" x2="48.26" y2="67.31" width="0.1524" layer="1"/>
-<wire x1="48.26" y1="67.31" x2="13.335" y2="67.31" width="0.1524" layer="1"/>
-<wire x1="13.335" y1="67.31" x2="11.43" y2="69.215" width="0.1524" layer="1"/>
-<wire x1="60.325" y1="62.865" x2="56.515" y2="62.865" width="0.1524" layer="1"/>
-<wire x1="56.515" y1="62.865" x2="50.165" y2="69.215" width="0.1524" layer="1"/>
+<wire x1="144.145" y1="57.785" x2="134.62" y2="48.26" width="0.1524" layer="1"/>
+<wire x1="134.62" y1="48.26" x2="5.08" y2="48.26" width="0.1524" layer="1"/>
 <wire x1="-3.81" y1="62.865" x2="11.43" y2="69.215" width="0" layer="19" extent="1-1"/>
 <wire x1="-19.05" y1="62.865" x2="-3.81" y2="62.865" width="0" layer="19" extent="1-1"/>
 <wire x1="-29.21" y1="69.215" x2="-19.05" y2="62.865" width="0" layer="19" extent="1-1"/>
+<wire x1="5.08" y1="48.26" x2="-3.81" y2="62.865" width="0" layer="19" extent="1-1"/>
 <wire x1="-67.945" y1="69.215" x2="-29.21" y2="69.215" width="0" layer="19" extent="1-1"/>
 <wire x1="-83.185" y1="62.865" x2="-67.945" y2="69.215" width="0" layer="19" extent="1-1"/>
@@
 </signal>
 <signal name="N$23">
+<contactref element="BCD2" pad="P$12"/>
+<contactref element="SR1" pad="P$8"/>
+<contactref element="SR1" pad="P$13"/>
+<contactref element="BCD3" pad="P$12"/>
+<wire x1="13.97" y1="74.295" x2="11.43" y2="76.835" width="0.1524" layer="16"/>
+<wire x1="47.625" y1="74.295" x2="13.97" y2="74.295" width="0.1524" layer="16"/>
+<contactref element="U$1" pad="GND@0"/>
 <contactref element="BCD4" pad="P$12"/>
 <contactref element="SR2" pad="P$8"/>
 <contactref element="BCD5" pad="P$12"/>
 <contactref element="SR2" pad="P$13"/>
+<wire x1="47.625" y1="74.295" x2="141.605" y2="57.785" width="0" layer="19" extent="16-16"/>
+<wire x1="-1.27" y1="55.245" x2="11.43" y2="76.835" width="0" layer="19" extent="1-1"/>
+<wire x1="-11.43" y1="62.865" x2="-1.27" y2="55.245" width="0" layer="19" extent="1-1"/>
+<wire x1="-29.21" y1="76.835" x2="-11.43" y2="62.865" width="0" layer="19" extent="1-1"/>
+<wire x1="-67.945" y1="76.835" x2="-29.21" y2="76.835" width="0" layer="19" extent="1-1"/>
+<wire x1="-80.645" y1="55.245" x2="-67.945" y2="76.835" width="0" layer="19" extent="1-1"/>
+<wire x1="-90.805" y1="62.865" x2="-80.645" y2="55.245" width="0" layer="19" extent="1-1"/>
+<wire x1="-108.585" y1="76.835" x2="-90.805" y2="62.865" width="0" layer="19" extent="1-1"/>
+</signal>
+<signal name="N$44">
+<contactref element="BCD0" pad="P$5"/>
+<contactref element="SR0" pad="P$16"/>
+<contactref element="U$1" pad="3V3@2"/>
+<contactref element="BCD1" pad="P$5"/>
+<contactref element="SR0" pad="P$10"/>
+<wire x1="145.415" y1="71.755" x2="93.345" y2="71.755" width="0.1524" layer="1"/>
+<wire x1="93.345" y1="71.755" x2="90.805" y2="69.215" width="0.1524" layer="1"/>
+<wire x1="154.305" y1="80.645" x2="145.415" y2="71.755" width="0.1524" layer="1"/>
+<wire x1="75.565" y1="62.865" x2="76.835" y2="64.135" width="0.1524" layer="1"/>
+<wire x1="85.725" y1="64.135" x2="76.835" y2="64.135" width="0.1524" layer="1"/>
+<wire x1="90.805" y1="69.215" x2="85.725" y2="64.135" width="0.1524" layer="1"/>
+<wire x1="76.835" y1="57.785" x2="77.47" y2="58.42" width="0.1524" layer="1"/>
+<wire x1="77.47" y1="60.96" x2="75.565" y2="62.865" width="0.1524" layer="1"/>
+<wire x1="50.165" y1="69.215" x2="61.595" y2="57.785" width="0.1524" layer="1"/>
+<wire x1="61.595" y1="57.785" x2="76.835" y2="57.785" width="0.1524" layer="1"/>
+<wire x1="77.47" y1="58.42" x2="77.47" y2="60.96" width="0.1524" layer="1"/>
+<wire x1="60.325" y1="62.865" x2="56.515" y2="62.865" width="0.1524" layer="1"/>
+<wire x1="56.515" y1="62.865" x2="50.165" y2="69.215" width="0.1524" layer="1"/>
+</signal>
+<signal name="N$45">
 <contactref element="BCD0" pad="P$12"/>
 <contactref element="SR0" pad="P$8"/>
@@
 <contactref element="SR0" pad="P$13"/>
 <contactref element="BCD1" pad="P$12"/>
-<contactref element="BCD2" pad="P$12"/>
-<contactref element="SR1" pad="P$8"/>
-<contactref element="SR1" pad="P$13"/>
-<contactref element="BCD3" pad="P$12"/>
 <wire x1="90.805" y1="76.835" x2="88.265" y2="74.295" width="0.1524" layer="16"/>
 <wire x1="88.265" y1="74.295" x2="52.705" y2="74.295" width="0.1524" layer="16"/>
@@
 <wire x1="67.945" y1="62.865" x2="66.675" y2="61.595" width="0.1524" layer="16"/>
 <wire x1="52.705" y1="74.295" x2="50.165" y2="76.835" width="0.1524" layer="16"/>
-<wire x1="50.165" y1="76.835" x2="47.625" y2="74.295" width="0.1524" layer="16"/>
-<wire x1="13.97" y1="74.295" x2="11.43" y2="76.835" width="0.1524" layer="16"/>
-<wire x1="47.625" y1="74.295" x2="13.97" y2="74.295" width="0.1524" layer="16"/>
 <via x="60.325" y="64.77" extent="1-16" drill="0.35"/>
 <wire x1="50.165" y1="76.835" x2="50.165" y2="74.295" width="0.1524" layer="1"/>
@@
 <wire x1="93.345" y1="74.295" x2="100.965" y2="74.295" width="0.1524" layer="1"/>
 <wire x1="100.965" y1="74.295" x2="102.87" y2="76.2" width="0.1524" layer="1"/>
-<wire x1="-1.27" y1="55.245" x2="11.43" y2="76.835" width="0" layer="19" extent="1-1"/>
-<wire x1="-11.43" y1="62.865" x2="-1.27" y2="55.245" width="0" layer="19" extent="1-1"/>
-<wire x1="-29.21" y1="76.835" x2="-11.43" y2="62.865" width="0" layer="19" extent="1-1"/>
-<wire x1="-67.945" y1="76.835" x2="-29.21" y2="76.835" width="0" layer="19" extent="1-1"/>
-<wire x1="-80.645" y1="55.245" x2="-67.945" y2="76.835" width="0" layer="19" extent="1-1"/>
-<wire x1="-90.805" y1="62.865" x2="-80.645" y2="55.245" width="0" layer="19" extent="1-1"/>
-<wire x1="-108.585" y1="76.835" x2="-90.805" y2="62.865" width="0" layer="19" extent="1-1"/>
 </signal>
 </signals>
