File: Hardware/KiCAD/NixieClock/NixieClock.sch (KiCad schematic (older format))
At the start: 3 parts, among them J0 39-29-6128

Commit message: Finished routing one complete stage... Now trying to make a kicad sch
Parts:
- removed J0, J? (x2): 39-29-6128, symbol Connector:39-29-6128
- added BCD0, BCD1, BCD2, BCD3, BCD4, BCD5: DM5441ADIP-16, NixieClock:DIP-16, symbol NixieClock-eagle-import:DM5441ADIP-16
- added SR0, SR1, SR2: SN74HC595NDIP-16, NixieClock:DIP-16, symbol NixieClock-eagle-import:SN74HC595NDIP-16
- added U$1: ESP12E_DEVKIT, NixieClock:ESP12E_DEVKIT, symbol NixieClock-eagle-import:ESP12E_DEVKIT
- added X0, X1, X2, X3, X4, X5: 5566-12, NixieClock:5566-12, symbol NixieClock-eagle-import:5566-12
Connections:
- wire segments 0 -> 176

Commit message: Progress
Parts:
- removed X0, X1, X2, X3, X4, X5: 5566-12, NixieClock:5566-12, symbol NixieClock-eagle-import:5566-12
- BCD0, BCD1, BCD2, BCD3, BCD4, BCD5: footprint NixieClock:DIP-16 -> NixieClock:DM7441A
- SR0, SR1, SR2: footprint NixieClock:DIP-16 -> NixieClock:SN74HC595
- U$1: footprint NixieClock:ESP12E_DEVKIT -> NixieClock:NODEMCU
